Commit message: normal looks

File: urdf/robot.urdf.xacro (robot description, xacro)
@@ -22,6 +22,6 @@
         <visual>
             <geometry><cylinder radius="0.08" length="0.05"/></geometry>
-            <origin xyz="0 0 0.25" rpy="0 0 0"/>
-            <material name="red">
+            <origin xyz="0 0 0.0" rpy="0 0 0"/>
+            <material name="green">
                 <color rgba="0 1 0 1"/>
             </material>
@@ -31,5 +31,5 @@
         <parent link="base_link"/>
         <child link="lidar_link"/>
-        <origin xyz="0 0 0.25"/>
+        <origin xyz="0 0 0.12"/>
     </joint>
     <xacro:macro name="wheel" params="name x y">
@@ -46,14 +46,17 @@
             <parent link="base_link"/>
             <child link="${name}"/>
-            <origin xyz="${x} ${y} 0.1" rpy="0 0 0"/>
+            <origin xyz="${x} ${y} -0.1" rpy="0 0 0"/>
             <axis xyz="0 1 0"/>
         </joint>
     </xacro:macro>
-    <xacro:wheel name="left_wheel" x="0" y="0.3"/>
-    <xacro:wheel name="right_wheel" x="0" y="-0.3"/>
+    <xacro:wheel name="left_wheel" x="0.1" y="0.3"/>
+    <xacro:wheel name="right_wheel" x="0.1" y="-0.3"/>
     <link name="caster_link">
         <visual>
             <geometry><sphere radius="0.05"/></geometry>
-            <origin xyz="-0.15 0 0.05"/>
+            <origin xyz="-0.1 0 0.0"/>
+            <material name="black">
+                <color rgba="0 0 0 1"/>
+            </material>
         </visual>
     </link>
@@ -61,5 +64,5 @@
         <parent link="base_link"/>
         <child link="caster_link"/>
-        <origin xyz="-0.15 0 0.05"/>
+        <origin xyz="-0.1 0 -0.1"/>
     </joint>
     <ros2_control name="MyRobotHardware" type="system">

Commit message: robot w gazebo

File: urdf/robot.urdf.xacro (robot description, xacro)
@@ -1,83 +1,146 @@
 <robot name="my_turtle" xmlns:xacro="http://ros.org/wiki/xacro">
-    <link name="base_link">
+  <!-- Gazebo plugin for ros2_control -->
+  <gazebo>
+    <plugin name="gazebo_ros2_control" filename="libgazebo_ros2_control.so"/>
+  </gazebo>
+  <link name="base_link">
     <visual>
-        <geometry>
-            <box size="0.4 0.6 0.2"/>
-        </geometry>
-        <material name="red">
-            <color rgba="1 0 0 0.7"/>
-        </material>
+      <geometry>
+        <box size="0.4 0.6 0.2"/>
+      </geometry>
+      <material name="red">
+        <color rgba="1 0 0 0.7"/>
+      </material>
     </visual>
     <collision>
-        <geometry>
+      <geometry>
         <box size="0.4 0.6 0.2"/>
-        </geometry>
+      </geometry>
     </collision>
     <inertial>
-        <mass value="10"/>
-        <inertia ixx="1e-3" ixy="0.0" ixz="0.0" iyy="1e-3" iyz="0.0" izz="1e-3"/>
+      <mass value="10"/>
+      <inertia ixx="0.1" ixy="0" ixz="0" iyy="0.1" iyz="0" izz="0.1"/>
     </inertial>
+  </link>
+  <link name="lidar_link">
+    <visual>
+      <geometry>
+        <cylinder radius="0.08" length="0.05"/>
+      </geometry>
+      <origin xyz="0 0 0.0" rpy="0 0 0"/>
+      <material name="green">
+        <color rgba="0 1 0 1"/>
+      </material>
+    </visual>
+    <collision>
+      <geometry>
+        <cylinder radius="0.08" length="0.05"/>
+      </geometry>
+    </collision>
+    <inertial>
+      <mass value="0.2"/>
+      <inertia ixx="0.001" ixy="0" ixz="0" iyy="0.001" iyz="0" izz="0.001"/>
+    </inertial>
+  </link>
+  <!-- LIDAR sensor plugin -->
+  <gazebo reference="lidar_link">
+    <sensor type="gpu_ray" name="lidar_sensor">
+      <update_rate>10</update_rate>
+      <ray>
+        <scan>
+          <horizontal>
+            <samples>720</samples>
+            <resolution>1</resolution>
+            <min_angle>-1.5708</min_angle>
+            <max_angle>1.5708</max_angle>
+          </horizontal>
+        </scan>
+        <range>
+          <min>0.1</min>
+          <max>10.0</max>
+        </range>
+      </ray>
+      <plugin name="gazebo_ros_laser" filename="libgazebo_ros_gpu_laser.so">
+        <ros_topic>/scan</ros_topic>
+        <frame_name>lidar_link</frame_name>
+      </plugin>
+    </sensor>
+  </gazebo>
+  <joint name="lidar_joint" type="fixed">
+    <parent link="base_link"/>
+    <child link="lidar_link"/>
+    <origin xyz="0 0 0.12"/>
+  </joint>
+  <xacro:macro name="wheel" params="name x y">
+    <link name="${name}">
+      <visual>
+        <geometry>
+          <cylinder radius="0.1" length="0.05"/>
+        </geometry>
+        <origin xyz="0 0 0" rpy="1.5708 0 0"/>
+        <material name="black">
+          <color rgba="0 0 0 1"/>
+        </material>
+      </visual>
+      <collision>
+        <geometry>
+          <cylinder radius="0.1" length="0.05"/>
+        </geometry>
+        <origin xyz="0 0 0" rpy="1.5708 0 0"/>
+      </collision>
+      <inertial>
+        <mass value="0.5"/>
+        <inertia ixx="0.001" iyy="0.001" izz="0.001" ixy="0" ixz="0" iyz="0"/>
+      </inertial>
     </link>
-    <link name="lidar_link">
-        <visual>
-            <geometry><cylinder radius="0.08" length="0.05"/></geometry>
-            <origin xyz="0 0 0.0" rpy="0 0 0"/>
-            <material name="green">
-                <color rgba="0 1 0 1"/>
-            </material>
-        </visual>
-    </link>
-    <joint name="lidar_joint" type="fixed">
-        <parent link="base_link"/>
-        <child link="lidar_link"/>
-        <origin xyz="0 0 0.12"/>
+    <joint name="${name}_joint" type="continuous">
+      <parent link="base_link"/>
+      <child link="${name}"/>
+      <origin xyz="${x} ${y} -0.1" rpy="0 0 0"/>
+      <axis xyz="0 1 0"/>
     </joint>
-    <xacro:macro name="wheel" params="name x y">
-        <link name="${name}">
-            <visual>
-                <geometry><cylinder radius="0.1" length="0.05"/></geometry>
-                <origin xyz="0 0 0" rpy="1.5708 0 0"/>
-                <material name="black">
-                    <color rgba="0 0 0 1"/>
-                </material>
-            </visual>
-        </link>
-        <joint name="${name}_joint" type="continuous">
-            <parent link="base_link"/>
-            <child link="${name}"/>
-            <origin xyz="${x} ${y} -0.1" rpy="0 0 0"/>
-            <axis xyz="0 1 0"/>
-        </joint>
-    </xacro:macro>
-    <xacro:wheel name="left_wheel" x="0.1" y="0.3"/>
-    <xacro:wheel name="right_wheel" x="0.1" y="-0.3"/>
-    <link name="caster_link">
-        <visual>
-            <geometry><sphere radius="0.05"/></geometry>
-            <origin xyz="-0.1 0 0.0"/>
-            <material name="black">
-                <color rgba="0 0 0 1"/>
-            </material>
-        </visual>
-    </link>
-    <joint name="caster_joint" type="fixed">
-        <parent link="base_link"/>
-        <child link="caster_link"/>
-        <origin xyz="-0.1 0 -0.1"/>
-    </joint>
-    <ros2_control name="MyRobotHardware" type="system">
+  </xacro:macro>
+  <xacro:wheel name="left_wheel" x="0.1" y="0.3"/>
+  <xacro:wheel name="right_wheel" x="0.1" y="-0.3"/>
+  <link name="caster_link">
+    <visual>
+      <geometry>
+        <sphere radius="0.05"/>
+      </geometry>
+      <origin xyz="-0.1 0 0.0"/>
+      <material name="black">
+        <color rgba="0 0 0 1"/>
+      </material>
+    </visual>
+    <collision>
+      <geometry>
+        <sphere radius="0.05"/>
+      </geometry>
+      <origin xyz="-0.1 0 0.0"/>
+    </collision>
+    <inertial>
+      <mass value="0.2"/>
+      <inertia ixx="0.0001" iyy="0.0001" izz="0.0001" ixy="0" ixz="0" iyz="0"/>
+    </inertial>
+  </link>
+  <joint name="caster_joint" type="fixed">
+    <parent link="base_link"/>
+    <child link="caster_link"/>
+    <origin xyz="-0.1 0 -0.1"/>
+  </joint>
+  <ros2_control name="MyRobotHardware" type="system">
     <hardware>
-        <plugin>fake_components/GenericSystem</plugin>
+      <plugin>fake_components/GenericSystem</plugin>
     </hardware>
     <joint name="left_wheel_joint">
-        <command_interface name="velocity"/>
-        <state_interface name="position"/>
-        <state_interface name="velocity"/>
+      <command_interface name="velocity"/>
+      <state_interface name="position"/>
+      <state_interface name="velocity"/>
     </joint>
     <joint name="right_wheel_joint">
-        <command_interface name="velocity"/>
-        <state_interface name="position"/>
-        <state_interface name="velocity"/>
+      <command_interface name="velocity"/>
+      <state_interface name="position"/>
+      <state_interface name="velocity"/>
     </joint>
-    </ros2_control>
+  </ros2_control>
 </robot>
